File: futuresight/futuresight.kicad_pcb (KiCad board)
At the start: 2 copper layers, 119.5 x 60 mm, 40 parts, among them J1 Conn_02x13_Odd_Even, J2 Conn_02x13_Odd_Even, J3 Conn_01x02, Q1 AO3401A, SW1 SW_Push, U1 TPS54360DDA

Commit message: updated -- pcb CAD firmware
Parts:
- moved C_IN1 48.2 mm to (175.2, 93.4)
- moved R_RT1 45.7 mm to (122.5, 95.3)
- moved Q1 38.6 mm to (177.0, 87.0)
- moved G*** 33.5 mm to (148.4, 88.6)
- moved F1 31.4 mm to (185.4, 87.2)
- moved C_OUT1 30.1 mm to (167.5, 108.0)
- moved C_OUT2 30.1 mm to (167.7, 112.2)
- moved D1 26.0 mm to (174.7, 101.1), turned to -90 degrees
- moved C_IN2 22.0 mm to (176.6, 78.3)
- moved D_BACKUP1 21.5 mm to (147.9, 74.5)
- moved R_SENSE2 21.2 mm to (129.4, 95.3)
- moved L1 19.4 mm to (158.7, 109.8), turned to -90 degrees
- moved U_MPU1 18.5 mm to (127.3, 74.9)
- moved C_BOOT1 15.2 mm to (122.6, 82.2)
- moved C_COMP1 15.2 mm to (122.6, 86.2)
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Routing:
- net C_boot_1: track 32.6 -> 139.5 mm, vias 2 -> 4
- net +5V_DUO: track 131.9 -> 211.0 mm, vias 1 -> 4
- net Net-(U1-RT/CLK): track 14.7 -> 88.0 mm
- net Net-(D_BACKUP1-A): track 107.1 -> 56.5 mm
- net +12V_PROT: track 79.3 -> 32.5 mm, vias 3 -> 1
- net MOSFET_Drain: track 49.0 -> 11.6 mm
- net +12V_RAW: track 50.2 -> 24.5 mm, vias 3 -> 0
- net I2C1_SCL: track 103.2 -> 79.6 mm, vias 0 -> 2
- net PWR_LOSS_GPIO: track 77.5 -> 98.4 mm, vias 1 -> 3
- net INT: track 26.2 -> 44.6 mm
- net GND: track 352.0 -> 333.7 mm, vias 14 -> 1
- net Net-(U1-COMP): track 41.2 -> 57.4 mm, vias 0 -> 2
- net U1_pin8: track 94.7 -> 79.0 mm, vias 0 -> 2
- net Net-(Q1-G): track 28.1 -> 43.5 mm, vias 0 -> 2
- net I2C1_SDA: track 65.1 -> 74.9 mm, vias 2 -> 3
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
Commit message: update ini. bom +pcb. change
Parts:
- C_OUT1, C_OUT2: footprint Capacitor_SMD:C_0805_2012Metric_Pad1.18x1.45mm_HandSolder -> Capacitor_SMD:C_1206_3216Metric_Pad1.33x1.80mm_HandSolder
Routing:
- net +5V_SYS: track 81.4 -> 78.2 mm
- removed copper zone on B.Cu, net GND
- removed copper zone on F.Cu, net GND
Changed lines of the file:
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@@
 		)
 	)
-	(footprint "Capacitor_SMD:C_0805_2012Metric_Pad1.18x1.45mm_HandSolder"
+	(footprint "Capacitor_SMD:C_1206_3216Metric_Pad1.33x1.80mm_HandSolder"
 		(layer "F.Cu")
 		(at 167.72 112.23)
-		(descr "Capacitor SMD 0805 (2012 Metric), square (rectangular) end terminal, IPC-7351 nominal with elongated pad for handsoldering. (Body size source: IPC-SM-782 page 76, https://www.pcb-3d.com/wordpress/wp-content/uploads/ipc-sm-782a_amendment_1_and_2.pdf, https://docs.google.com/spreadsheets/d/1BsfQQcO9C6DZCsRaXUlFlo91Tg2WpOkGARC1WS5S8t0/edit?usp=sharing)")
+		(descr "Capacitor SMD 1206 (3216 Metric), square (rectangular) end terminal, IPC-7351 nominal with elongated pad for handsoldering. (Body size source: IPC-SM-782 page 76, https://www.pcb-3d.com/wordpress/wp-content/uploads/ipc-sm-782a_amendment_1_and_2.pdf)")
 		(tags "capacitor handsolder")
 		(property "Reference" "C_OUT2"
-			(at 0 -1.68 0)
+			(at 0 -1.85 0)
 			(layer "F.SilkS")
 			(effects
@@
 		)
 		(property "Value" "22µF"
-			(at 0 1.68 0)
+			(at 0 1.85 0)
 			(layer "F.Fab")
 			(effects
@@
 			)
 		)
-		(property "Description" "22µF 16V X5R Ceramic Cap"
+		(property "Description" "22µF 16V X7R Ceramic Cap"
 			(at 0 0 0)
 			(layer "F.Fab")
@@
 		(duplicate_pad_numbers_are_jumpers no)
 		(fp_line
-			(start -0.261252 -0.735)
-			(end 0.261252 -0.735)
+			(start -0.711252 -0.91)
+			(end 0.711252 -0.91)
 			(stroke
 				(width 0.12)
@@
 		)
 		(fp_line
-			(start -0.261252 0.735)
-			(end 0.261252 0.735)
+			(start -0.711252 0.91)
+			(end 0.711252 0.91)
 			(stroke
 				(width 0.12)
@@
 		)
 		(fp_rect
-			(start -1.88 -0.98)
-			(end 1.88 0.98)
+			(start -2.48 -1.15)
+			(end 2.48 1.15)
 			(stroke
 				(width 0.05)
@@
 		)
 		(fp_rect
-			(start -1 -0.625)
-			(end 1 0.625)
+			(start -1.6 -0.8)
+			(end 1.6 0.8)
 			(stroke
 				(width 0.1)
@@
 			(effects
 				(font
-					(size 0.5 0.5)
-					(thickness 0.08)
+					(size 0.8 0.8)
+					(thickness 0.12)
 				)
 			)
 		)
 		(pad "1" smd roundrect
-			(at -1.0375 0)
-			(size 1.175 1.45)
+			(at -1.5625 0)
+			(size 1.325 1.8)
 			(layers "F.Cu" "F.Mask" "F.Paste")
-			(roundrect_rratio 0.212766)
+			(roundrect_rratio 0.188679)
 			(net "+5V_SYS")
 			(pintype "passive")
 		)
 		(pad "2" smd roundrect
-			(at 1.0375 0)
-			(size 1.175 1.45)
+			(at 1.5625 0)
+			(size 1.325 1.8)
 			(layers "F.Cu" "F.Mask" "F.Paste")
-			(roundrect_rratio 0.212766)
+			(roundrect_rratio 0.188679)
 			(net "GND")
 			(pintype "passive")
 		)
 		(embedded_fonts no)
-		(model "${KICAD10_3DMODEL_DIR}/Capacitor_SMD.3dshapes/C_0805_2012Metric.step"
+		(model "${KICAD10_3DMODEL_DIR}/Capacitor_SMD.3dshapes/C_1206_3216Metric.step"
 			(offset
 				(xyz 0 0 0)
@@
 		)
 	)
-	(footprint "Capacitor_SMD:C_0805_2012Metric_Pad1.18x1.45mm_HandSolder"
+	(footprint "Capacitor_SMD:C_1206_3216Metric_Pad1.33x1.80mm_HandSolder"
 		(layer "F.Cu")
 		(at 167.47 107.98)
-		(descr "Capacitor SMD 0805 (2012 Metric), square (rectangular) end terminal, IPC-7351 nominal with elongated pad for handsoldering. (Body size source: IPC-SM-782 page 76, https://www.pcb-3d.com/wordpress/wp-content/uploads/ipc-sm-782a_amendment_1_and_2.pdf, https://docs.google.com/spreadsheets/d/1BsfQQcO9C6DZCsRaXUlFlo91Tg2WpOkGARC1WS5S8t0/edit?usp=sharing)")
+		(descr "Capacitor SMD 1206 (3216 Metric), square (rectangular) end terminal, IPC-7351 nominal with elongated pad for handsoldering. (Body size source: IPC-SM-782 page 76, https://www.pcb-3d.com/wordpress/wp-content/uploads/ipc-sm-782a_amendment_1_and_2.pdf)")
 		(tags "capacitor handsolder")
 		(property "Reference" "C_OUT1"
-			(at 0 -1.68 0)
+			(at 0 -1.85 0)
 			(layer "F.SilkS")
 			(effects
@@
 		)
 		(property "Value" "22µF"
-			(at 0 1.68 0)
+			(at 0 1.85 0)
 			(layer "F.Fab")
 			(effects
@@
 			)
 		)
-		(property "Description" "22µF 16V X5R Ceramic Cap"
+		(property "Description" "22µF 16V X7R Ceramic Cap"
 			(at 0 0 0)
 			(layer "F.Fab")
@@
 		(duplicate_pad_numbers_are_jumpers no)
 		(fp_line
-			(start -0.261252 -0.735)
-			(end 0.261252 -0.735)
+			(start -0.711252 -0.91)
+			(end 0.711252 -0.91)
 			(stroke
 				(width 0.12)
@@
 		)
 		(fp_line
-			(start -0.261252 0.735)
-			(end 0.261252 0.735)
+			(start -0.711252 0.91)
+			(end 0.711252 0.91)
 			(stroke
 				(width 0.12)
@@
 		)
 		(fp_rect
-			(start -1.88 -0.98)
-			(end 1.88 0.98)
+			(start -2.48 -1.15)
+			(end 2.48 1.15)
 			(stroke
 				(width 0.05)
@@
 		)
 		(fp_rect
-			(start -1 -0.625)
-			(end 1 0.625)
+			(start -1.6 -0.8)
+			(end 1.6 0.8)
 			(stroke
 				(width 0.1)
@@
 			(effects
 				(font
-					(size 0.5 0.5)
-					(thickness 0.08)
+					(size 0.8 0.8)
+					(thickness 0.12)
 				)
 			)
 		)
 		(pad "1" smd roundrect
-			(at -1.0375 0)
-			(size 1.175 1.45)
+			(at -1.5625 0)
+			(size 1.325 1.8)
 			(layers "F.Cu" "F.Mask" "F.Paste")
-			(roundrect_rratio 0.212766)
+			(roundrect_rratio 0.188679)
 			(net "+5V_SYS")
 			(pintype "passive")
 		)
 		(pad "2" smd roundrect
-			(at 1.0375 0)
-			(size 1.175 1.45)
+			(at 1.5625 0)
+			(size 1.325 1.8)
 			(layers "F.Cu" "F.Mask" "F.Paste")
-			(roundrect_rratio 0.212766)
+			(roundrect_rratio 0.188679)
 			(net "GND")
 			(pintype "passive")
 		)
 		(embedded_fonts no)
-		(model "${KICAD10_3DMODEL_DIR}/Capacitor_SMD.3dshapes/C_0805_2012Metric.step"
+		(model "${KICAD10_3DMODEL_DIR}/Capacitor_SMD.3dshapes/C_1206_3216Metric.step"
 			(offset
 				(xyz 0 0 0)
@@
 		(sheetname "/duos_interface/")
 		(sheetfile "duos_interface.kicad_sch")
+		(units
+			(unit
+				(name "A")
+				(pins "1" "3" "5" "7" "9" "11" "13" "15" "17" "19" "21" "23" "25" "2"
+					"4" "6" "8" "10" "12" "14" "16" "18" "20" "22" "24" "26"
+				)
+			)
+		)
 		(attr through_hole)
 		(duplicate_pad_numbers_are_jumpers no)
@@
 	)
 	(segment
-		(start 168.775 121.25)
-		(end 167.15 119.625)
-		(width 1.3)
-		(layer "F.Cu")
-		(net "GND")
-	)
-	(segment
-		(start 167.15 119.625)
-		(end 167.15 114.5625)
-		(width 1.3)
-		(layer "F.Cu")
-		(net "GND")
-	)
-	(segment
 		(start 167.2525 102.58)
 		(end 162.07 97.3975)
@@
 	)
 	(segment
-		(start 168.5075 107.98)
-		(end 168.5075 104.38)
-		(width 1.3)
-		(layer "F.Cu")
-		(net "GND")
-	)
-	(segment
-		(start 167.15 114.5625)
-		(end 168.7575 112.955)
+		(start 167.15 119.625)
+		(end 167.15 114.3625)
 		(width 1.3)
 		(layer "F.Cu")
@@
 	)
 	(segment
+		(start 167.15 114.3625)
+		(end 169.2825 112.23)
+		(width 1.3)
+		(layer "F.Cu")
+		(net "GND")
+	)
+	(segment
 		(start 130.305 96.955)
 		(end 130.305 95.27)
@@
 	)
 	(segment
+		(start 169.2825 108.23)
+		(end 169.0325 107.98)
+		(width 1.3)
+		(layer "F.Cu")
+		(net "GND")
+	)
+	(segment
 		(start 124.16 97.86)
 		(end 129.52 97.86)
@@
 	)
 	(segment
+		(start 169.0325 107.98)
+		(end 169.0325 104.905)
+		(width 1.3)
+		(layer "F.Cu")
+		(net "GND")
+	)
+	(segment
 		(start 130.825 95.27)
 		(end 136.015 90.08)
@@
 	)
 	(segment
+		(start 169.0325 104.905)
+		(end 168.5075 104.38)
+		(width 1.3)
+		(layer "F.Cu")
+		(net "GND")
+	)
+	(segment
 		(start 95.715 78.115)
 		(end 98.255 78.115)
@@
 	)
 	(segment
-		(start 168.7575 112.955)
-		(end 168.7575 112.23)
-		(width 1.3)
-		(layer "F.Cu")
-		(net "GND")
-	)
-	(segment
 		(start 174.7 103.245)
 		(end 180.215 103.245)
@@
 	)
 	(segment
+		(start 169.2825 112.23)
+		(end 169.2825 108.23)
+		(width 1.3)
+		(layer "F.Cu")
+		(net "GND")
+	)
+	(segment
 		(start 129.28 73.63)
 		(end 129.772764 73.63)
@@
 	)
 	(segment
+		(start 168.775 121.25)
+		(end 167.15 119.625)
+		(width 1.3)
+		(layer "F.Cu")
+		(net "GND")
+	)
+	(segment
 		(start 88.285 75.575)
 		(end 89.46 76.75)
@@
 	)
 	(segment
-		(start 168.7575 112.23)
-		(end 168.7575 108.23)
-		(width 1.3)
-		(layer "F.Cu")
-		(net "GND")
-	)
-	(segment
 		(start 89.46 76.75)
 		(end 90.825 78.115)
@@
 	)
 	(segment
-		(start 168.7575 108.23)
-		(end 168.5075 107.98)
-		(width 1.3)
-		(layer "F.Cu")
-		(net "GND")
-	)
-	(segment
 		(start 160.47 93.17)
 		(end 161.73 94.43)
@@
 	)
 	(segment
-		(start 166.4325 107.98)
-		(end 166.4325 111.98)
-		(width 1.3)
-		(layer "F.Cu")
-		(net "+5V_SYS")
-	)
-	(segment
-		(start 158.66 112.58)
-		(end 166.3325 112.58)
-		(width 1.3)
-		(layer "F.Cu")
-		(net "+5V_SYS")
-	)
-	(segment
 		(start 161.3475 117.14)
 		(end 161.56 117.3525)
@@
 	)
 	(segment
-		(start 166.4325 111.98)
-		(end 166.6825 112.23)
+		(start 161.3475 117.14)
+		(end 161.3475 115.2675)
 		(width 1.3)
 		(layer "F.Cu")
@@
 	)
 	(segment
-		(start 166.3325 112.58)
-		(end 166.6825 112.23)
+		(start 166.1575 108.23)
+		(end 165.9075 107.98)
 		(width 1.3)
 		(layer "F.Cu")
@@
 	)
 	(segment
+		(start 166.1575 112.23)
+		(end 166.1575 108.23)
+		(width 1.3)
+		(layer "F.Cu")
+		(net "+5V_SYS")
+	)
+	(segment
 		(start 143.45 109.86)
 		(end 143.69 110.1)
@@
 	)
 	(segment
-		(start 161.56 117.3525)
-		(end 166.3325 112.58)
+		(start 164.385 112.23)
+		(end 166.1575 112.23)
 		(width 1.3)
 		(layer "F.Cu")
@@
 		(net "+5V_SYS")
 	)
+	(segment
+		(start 161.3475 115.2675)
+		(end 158.66 112.58)
+		(width 1.3)
+		(layer "F.Cu")
+		(net "+5V_SYS")
+	)
+	(segment
+		(start 161.3475 115.2675)
+		(end 164.385 112.23)
+		(width 1.3)
+		(layer "F.Cu")
+		(net "+5V_SYS")
+	)
 	(via
 		(at 134.17 93.22)
@@
 			)
 		)
-	)
-	(zone
-		(net "GND")
-		(layers "F.Cu" "B.Cu")
-		(hatch edge 0.5)
-		(connect_pads
-			(clearance 0.5)
-		)
-		(min_thickness 0.25)
-		(fill yes
-			(thermal_gap 0.5)
-			(thermal_bridge_width 0.5)
-			(island_removal_mode 0)
-		)
-		(polygon
-			(pts
-				(xy 193.98 63.67) (xy 197.09 130.22) (xy 62.05 127.7) (xy 65.73 63.28)
-			)
-		)
