File: futuresight-pcb/safe_shut.kicad_sch (KiCad schematic)
At the start: 6 parts

Commit message: update pcb path
Parts:
- C_SUPER1: footprint Capacitor_THT:CP_Radial_D13.0mm_P5.00mm -> Capacitor_THT:CP_Radial_D24.0mm_P10.00mm_SnapIn
Changed lines of the file:
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@@
 			)
 		)
-		(property "Footprint" "Capacitor_THT:CP_Radial_D13.0mm_P5.00mm"
+		(property "Footprint" "Capacitor_THT:CP_Radial_D24.0mm_P10.00mm_SnapIn"
 			(at 78.74 33.02 0)
 			(hide yes)
